File: VAST.sch (EAGLE design)
At the start: 5 parts, among them U2 MPL3115A2

Commit message: Add files via upload
Parts:
- removed B1: TEENSY-3.1NOSILK, SparkFun-Boards:TEENSY-3.1NOSILK
- removed U2: MPL3115A2, SparkFun-Sensors:MPL3115A2
- added J4: (no value), SparkFun-Connectors:CONN_04POLAR
- added U$1: TEENSY_3.1_BASIC, Teensy_3_Series_Board_v1.0:TEENSY_3.1_BASIC
Connections:
- removed net N$10: B1.7/RX3
- removed net N$11: B1.8/TX3
- removed net N$12: B1.9*/RX2
- removed net N$14: B1.GND
- removed net N$16: B1.3.3V
- removed net N$18: B1.VIN, J1.1, J1.2, J2.1, J2.2, R1.1, U2.VDD
- removed net N$5: B1.2, R1.2
- removed net N$6: B1.A4/18/SDA0, U2.SDA
- removed net N$7: B1.A5/19/SCL0, U2.SCL
- removed net N$8: B1.0/RX1
- removed net N$9: B1.1/TX1
- net N$1: now also J1.2, J2.2, R1.1, U$1.2; no longer B1.13/SCK
- net N$13: now also J4.1, U$1.GND; no longer B1.GND1, U2.GND
- net N$2: now also J1.1, J2.1, J4.2, R1.2, U$1.3.3V; no longer B1.12/DIN
- net N$3: now also J4.3, U$1.18/A4/T/SDA0; no longer B1.11/DOUT
- net N$4: now also J4.4, U$1.19/A5/T/SCL0; no longer B1.10*/TX2/CS

Commit message: Add files via upload
Updated board with ground VIA and Two Test Pads
Parts:
- added PAD1, PAD3: (no value), wirepad:SMD5
Connections:
- net N$1: now also PAD1.P
- net N$2: now also PAD3.P
Changed lines of the file:
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@@
 <part name="U$1" library="Teensy_3_Series_Board_v1.0" deviceset="TEENSY_3.1_BASIC" device=""/>
 <part name="J4" library="SparkFun-Connectors" deviceset="CONN_04" device="POLAR"/>
+<part name="PAD1" library="wirepad" library_urn="urn:adsk.eagle:library:412" deviceset="SMD5" device="" package3d_urn="urn:adsk.eagle:package:30841/1"/>
+<part name="PAD3" library="wirepad" library_urn="urn:adsk.eagle:library:412" deviceset="SMD5" device="" package3d_urn="urn:adsk.eagle:package:30841/1"/>
 </parts>
 <sheets>
@@
 <attribute name="VALUE" x="33.02" y="25.654" size="1.778" layer="96" font="vector"/>
 <attribute name="NAME" x="33.02" y="41.148" size="1.778" layer="95" font="vector"/>
+</instance>
+<instance part="PAD1" gate="1" x="22.86" y="60.96" smashed="yes">
+<attribute name="NAME" x="21.717" y="62.8142" size="1.778" layer="95"/>
+<attribute name="VALUE" x="21.717" y="57.658" size="1.778" layer="96"/>
+</instance>
+<instance part="PAD3" gate="1" x="142.24" y="88.9" smashed="yes" rot="R270">
+<attribute name="NAME" x="144.0942" y="90.043" size="1.778" layer="95" rot="R270"/>
+<attribute name="VALUE" x="138.938" y="90.043" size="1.778" layer="96" rot="R270"/>
 </instance>
 </instances>
@@
 <pinref part="U$1" gate="G$1" pin="2"/>
 <wire x1="58.42" y1="76.2" x2="88.9" y2="76.2" width="0.1524" layer="91"/>
+<pinref part="PAD1" gate="1" pin="P"/>
+<wire x1="43.18" y1="60.96" x2="25.4" y2="60.96" width="0.1524" layer="91"/>
+<junction x="43.18" y="60.96"/>
 </segment>
 </net>
@@
 <junction x="58.42" y="33.02"/>
 <pinref part="J4" gate="J1" pin="2"/>
+<pinref part="PAD3" gate="1" pin="P"/>
+<wire x1="142.24" y1="78.74" x2="142.24" y2="86.36" width="0.1524" layer="91"/>
+<junction x="142.24" y="78.74"/>
 </segment>
 </net>
@@
 </schematic>
 </drawing>
+<compatibility>
+<note version="8.2" severity="warning">
+Since Version 8.2, EAGLE supports online libraries. The ids
+of those online libraries will not be understood (or retained)
+with this version.
+</note>
+<note version="8.3" severity="warning">
+Since Version 8.3, EAGLE supports URNs for individual library
+assets (packages, symbols, and devices). The URNs of those assets
+will not be understood (or retained) with this version.
+</note>
+<note version="8.3" severity="warning">
+Since Version 8.3, EAGLE supports the association of 3D packages
+with devices in libraries, schematics, and board files. Those 3D
+packages will not be understood (or retained) with this version.
+</note>
+</compatibility>
 </eagle>
